File: rag/spi_auto.kicad_sch (KiCad schematic)
At the start: 25 parts, among them U1 STM32L476JGYxP, U2 LSM6DSM

Commit message: Close footprint hallucination: resolver reads authoritative footprint from KiCad symbol, wins over LLM netlist value (Part 2)
Parts:
- U1: footprint (none) -> Package_CSP:ST_WLCSP-72_Die415
- U2: footprint (none) -> Package_LGA:LGA-14_3x2.5mm_P0.5mm_LayoutBorder3x4y
